Commit message: new file:   launch/robot_control.launch 	modified:   launch/robot_gazebo.launch 	modified:   robot/camera.xacro 	new file:   robot/gazebo_control.xacro 	modified:   robot/lidar.xacro 	modified:   robot/lidar2.xacro 	modified:   robot/robot.urdf.xacro 	modified:   robot/robot_base.xacro
	deleted:    aula_setup.bash

File: robot/camera.xacro (robot description, xacro)
@@ -4,5 +4,5 @@
         <parent link="corpo_link"/>
         <child link="camera_link"/>
-        <origin xyz="0.305 0 0.08" rpy="0 0 0"/>
+        <origin xyz="${tamanho_x/2} 0 ${tamanho_z}" rpy="0 0 0"/>
     </joint>
     <link name="camera_link">
@@ -19,8 +19,7 @@
         <origin xyz="0 0 0" rpy="${-pi/2} 0 ${-pi/2}"/>
     </joint>
-    <link name="camera_link_optical"></link>
     <gazebo reference="camera_link">
-        <material>Gazebo/Red</material>
-        <sensor name="camera" type="camera">
+        <material>Gazebo/White</material>
+        <sensor name="camera_sensor" type="camera">
             <pose> 0 0 0 0 0 0 </pose>
             <visualize>true</visualize>
@@ -39,5 +38,5 @@
             </camera>
             <plugin name="camera_controller" filename="libgazebo_ros_camera.so">
-                <frame_name>camera_link_optical</frame_name>
+                <frame_name>camera_link</frame_name>
             </plugin>
         </sensor>

File: robot/lidar.xacro (robot description, xacro)
@@ -4,5 +4,5 @@
         <parent link="corpo_link"/>
         <child link="laser_frame"/>
-        <origin xyz="0 0 ${tamanho_z/2+0.5}" rpy="0 0 0"/>
+        <origin xyz="0 0 0" rpy="0 0 0"/>
     </joint>
     <link name="laser_frame">
@@ -41,5 +41,5 @@
                 </range>
             </ray>
-            <plugin name="laser_controller" filename="libgazebo_ros_laser.so">
+            <plugin name="laser_controller" filename="libgazebo_ros_ray_sensor.so">
                 <ros>
                     <argument>~/out:=scan</argument>

File: robot/lidar2.xacro (robot description, xacro)
@@ -4,5 +4,5 @@
         <parent link="corpo_link"/>
         <child link="laser_frame"/>
-        <origin xyz="0 0 ${tamanho_z/2+0.5}" rpy="0 0 0"/>
+        <origin xyz="0 0 ${tamanho_z/2+0.01}" rpy="0 0 0"/>
     </joint>
     <link name="laser_frame">
@@ -27,26 +27,22 @@
             <pose>0 0 0 0 1.57079633 0</pose>
             <ray>
-              <scan>
-                <horizontal>
-                    <samples>360</samples>
-                    <resolution>1</resolution>
-                    <min_angle>-${pi}</min_angle>
-                    <max_angle>${pi}</max_angle>
-                </horizontal>
-              </scan>
-              <range>
-                <min>0.06</min> <!-- do not change: use min_distance (below) for realistic behavior (smaller values cause issues) -->
-                <max>10</max>   <!-- do not change: use min_distance (below) for realistic behavior (bigger values cause issues) -->
-                <resolution>0.01</resolution>
-              </range>
-              <noise>
-                <type>gaussian</type>
-                <mean>0.0</mean>
-                <stddev>0.02</stddev>
-              </noise>
+                <scan>
+                  <horizontal>
+                      <samples>360</samples>
+                      <resolution>1</resolution>
+                      <min_angle>-${pi}</min_angle>
+                      <max_angle>${pi}</max_angle>
+                  </horizontal>
+                </scan>
+                <range>
+                  <min>0.06</min> <!-- do not change: use min_distance (below) for realistic behavior (smaller values cause issues) -->
+                  <max>10</max>   <!-- do not change: use min_distance (below) for realistic behavior (bigger values cause issues) -->
+                </range>
             </ray>
-            <plugin name="laser_gazebo" filename="libgazebo_ros_laser.so" />
-            <always_on>1</always_on>
-            <update_rate>30</update_rate>
+            <plugin name="laser_gazebo" filename="libgazebo_ros_laser.so">
+                <topicName>/scan</topicName>
+                <frameName>laser_frame</frameName>
+            </plugin>
+            <update_rate>10</update_rate>
             <visualize>true</visualize>
         </sensor>

File: robot/robot.urdf.xacro (robot description, xacro)
@@ -2,6 +2,7 @@
 <robot name="robo" xmlns:xacro="http://www.ros.org/wiki/xacro">
     <xacro:include filename="robot_base.xacro"/>
+    <xacro:include filename="gazebo_control.xacro"/>
     <!-- <xacro:include filename="camera.xacro"/> -->
-    <xacro:include filename="lidar.xacro"/>
+    <xacro:include filename="lidar2.xacro"/>
     <!-- <xacro:include filename="kinetic.xacro"/> -->
 </robot>

File: robot/robot_base.xacro (robot description, xacro)
@@ -42,5 +42,21 @@
       </xacro:inertial_box>
   </link>
+  <gazebo reference="corpo_link">
+    <material>Gazebo/Red</material>
+  </gazebo>
   <!-- roda esquerda -->
+  <joint name="debug_joint" type="fixed">
+    <origin xyz="0.0 0.0 0.0" rpy="0.0 0.0 0.0"/>
+    <parent link="roda_esquerda_link"/>
+    <child link="debug_box"/>
+  </joint>
+  <link name="debug_box">
+    <visual>
+      <geometry>
+        <box size="0.05 0.05 0.05"/>
+      </geometry>
+      <material name="blue"/>
+    </visual>
+  </link>
   <joint name="roda_esquerda_joint" type="continuous">
     <parent link="base_link"/>
@@ -65,10 +81,26 @@
     </xacro:inertial_cylinder>
   </link>
+  <gazebo reference="roda_esquerda_link">
+    <material>Gazebo/Blue</material>
+  </gazebo>
   <!-- roda direita -->
+  <joint name="debug_direita_joint" type="fixed">
+    <origin xyz="0.0 0.0 0.0" rpy="0.0 0.0 0.0"/>
+    <parent link="roda_direita_link"/>
+    <child link="debug_box_2"/>
+  </joint>
+  <link name="debug_box_2">
+    <visual>
+      <geometry>
+        <box size="0.05 0.05 0.05"/>
+      </geometry>
+      <material name="blue"/>
+    </visual>
+  </link>
   <joint name="roda_direita_joint" type="continuous">
     <parent link="base_link"/>
     <child link="roda_direita_link"/>
     <origin xyz="-${tamanho_x/2+0.05} -${tamanho_y/2} -${tamanho_z/2}" rpy="${pi/2} 0.0 0.0"/>
-    <axis xyz="0.0 0.0 1.0"/>
+    <axis xyz="0.0 0.0 -1.0"/>
   </joint>
   <link name="roda_direita_link">
@@ -88,4 +120,7 @@
     </xacro:inertial_cylinder>
   </link>
+  <gazebo reference="roda_direita_link">
+    <material>Gazebo/Blue</material>
+  </gazebo>
   <!-- bolinha -->
   <joint name="bolinha_joint" type="fixed">
@@ -110,3 +145,8 @@
     </xacro:inertial_sphere>
   </link>
+  <gazebo reference="bolinha_link">
+    <material>Gazebo/Black</material>
+    <mu1 value="0.001"/>
+    <mu2 value="0.001"/>
+  </gazebo>
 </robot>
