Commit message: new file:   robot/camera2.xacro 	new file:   robot/depth_camera.xacro 	modified:   robot/kinetic.xacro 	deleted:    robot/lidar.xacro 	modified:   robot/lidar2.xacro 	modified:   robot/robot.urdf.xacro
	deleted:    aula_setup.bash

File: robot/lidar2.xacro (robot description, xacro)
@@ -11,5 +11,5 @@
                 <cylinder radius="0.05" length="0.04"/>
             </geometry>
-            <material name="red"/>
+            <material name="white"/>
         </visual>
         <collision>
@@ -23,5 +23,5 @@
     </link>
     <gazebo reference="laser_frame">
-        <material>Gazebo/Red</material>
+        <material>Gazebo/White</material>
         <sensor name="laser" type="ray">
             <pose>0 0 0 0 1.57079633 0</pose>

File: robot/robot.urdf.xacro (robot description, xacro)
@@ -3,6 +3,7 @@
     <xacro:include filename="robot_base.xacro"/>
     <xacro:include filename="gazebo_control.xacro"/>
-    <!-- <xacro:include filename="camera.xacro"/> -->
-    <xacro:include filename="lidar2.xacro"/>
-    <!-- <xacro:include filename="kinetic.xacro"/> -->
+    <!-- <xacro:include filename="camera2.xacro"/> -->
+    <!-- <xacro:include filename="depth_camera.xacro"/> -->
+    <!-- <xacro:include filename="lidar2.xacro"/> -->
+    <xacro:include filename="kinetic.xacro"/>
 </robot>
