Commit message: modified:   robot/camera2.xacro 	modified:   robot/kinetic.xacro 	modified:   robot/lidar2.xacro 	modified:   robot/robot.urdf.xacro 	deleted:    aula_setup.bash

File: robot/camera2.xacro (robot description, xacro)
@@ -14,5 +14,4 @@
         </visual>
     </link>
-    <!--
     <joint name="camera_optical_joint" type="fixed">
         <parent link="camera_link"/>
@@ -20,6 +19,5 @@
         <origin xyz="0 0 0" rpy="${-pi/2} 0 ${-pi/2}"/>
     </joint>
-    -->
-    <!-- <link name="camera_link_optical"></link> -->
+    <link name="camera_link_optical"></link>
     <gazebo reference="camera_link">
         <material>Gazebo/White</material>
@@ -41,5 +39,5 @@
             </camera>
             <plugin name="camera_controller" filename="libgazebo_ros_camera.so">
-                <frame_name>camera_link</frame_name>
+                <frame_name>camera_link_optical</frame_name>
             </plugin>
         </sensor>

File: robot/kinetic.xacro (robot description, xacro)
@@ -1,57 +1,69 @@
 <?xml version="1.0"?>
 <robot xmlns:xacro="http://www.ros.org/wiki/xacro" >
+  <joint name="kinetic_joint" type="fixed">
+    <origin xyz="${tamanho_x/2} 0 0" rpy="0.0 0.0 0.0"/>
+    <parent link="corpo_link"/>
+    <child link="kinetic_link"/>
+  </joint>
   <link name="kinetic_link">
     <visual>
-      <origin xyz="0.0 0.0 0.0" rpy="0.0 0.0 0.0"/>
+      <material name="white"/>
+      <origin xyz="0.0 0.0 0.0" rpy="${pi} 0.0 0.0"/>
       <geometry>
-        <box size="0.0 0.0 0.0"/>
+        <box size="0.05 0.05 0.05"/>
       </geometry>
     </visual>
   </link>
-  <joint name="kinetic_joint" type="fixed">
-    <origin xyz="-${tamanho_x/2} ${tamanho_y/3} 0.0" rpy="0.0 0.0 0.0"/>
-    <parent link="corpo_link"/>
-    <child link="kinetic_link"/>
-  </joint>
-  <sensor name="camera" type="depth">
-    <update_rate>0<update_rate>
-    <camera>
-      <horizontal_fov>1.047198</horizontal_fov>
-      <image>
-        <width>640</width>
-        <height>480</height>
-        <format>R8G8B8</format>
-      </image>
-      <clip>
-        <near>0.05</near>
-        <far>3</far>
-      </clip>
-    </camera>
-    <plugin name="camera_plugin" filename="libgazebo_ros_openni_kinect.so">
-        <baseline>0.2</baseline>
-        <alwaysOn>true</alwaysOn>
-        <!-- Keep this zero, update_rate in the parent <sensor> tag
-          will control the frame rate. -->
-        <updateRate>0.0</updateRate>
-        <cameraName>camera_ir</cameraName>
-        <imageTopicName>/agent/camera/color/image_raw</imageTopicName>
-        <cameraInfoTopicName>/agent/camera/color/camera_info</cameraInfoTopicName>
-        <depthImageTopicName>/agent/camera/depth/image_raw</depthImageTopicName>
-        <depthImageCameraInfoTopicName>/agent/camera/depth/camera_info</depthImageCameraInfoTopicName>
-        <pointCloudTopicName>/agent/camera/depth/points</pointCloudTopicName>
-        <frameName>camera_link</frameName>
-        <pointCloudCutoff>0.5</pointCloudCutoff>
-        <pointCloudCutoffMax>3.0</pointCloudCutoffMax>
-        <distortionK1>0</distortionK1>
-        <distortionK2>0</distortionK2>
-        <distortionK3>0</distortionK3>
-        <distortionT1>0</distortionT1>
-        <distortionT2>0</distortionT2>
-        <CxPrime>0</CxPrime>
-        <Cx>0</Cx>
-        <Cy>0</Cy>
-        <focalLength>0</focalLength>
-        <hackBaseline>0</hackBaseline>
-    </plugin>
-  </sensor>
+  <joint name="dumb_kinetic_joint" type="fixed">
+        <parent link="kinetic_link"/>
+        <child link="dumb_kinetic"/>
+        <origin xyz="0 0 0" rpy="${-pi/2} 0 ${-pi/2}"/>
+    </joint>
+  <link name="dumb_kinetic">
+  </link>
+  <gazebo reference='kinetic_link'>
+    <material>Gazebo/White</material>
+    <sensor name="camera" type="depth">
+      <update_rate>10</update_rate>
+      <camera>
+        <horizontal_fov>1.047198</horizontal_fov>
+        <image>
+          <width>640</width>
+          <height>480</height>
+          <!-- <format>R8G8B8</format> -->
+          <format>B8G8R8</format>
+        </image>
+        <clip>
+          <near>0.05</near>
+          <far>3</far>
+        </clip>
+      </camera>
+      <plugin name="camera_plugin" filename="libgazebo_ros_openni_kinect.so">
+          <baseline>0.2</baseline>
+          <alwaysOn>true</alwaysOn>
+          <!-- Keep this zero, update_rate in the parent <sensor> tag
+            will control the frame rate. -->
+          <updateRate>0.0</updateRate>
+          <cameraName>camera_ir</cameraName>
+          <imageTopicName>/agent/camera/color/image_raw</imageTopicName>
+          <cameraInfoTopicName>/agent/camera/color/camera_info</cameraInfoTopicName>
+          <depthImageTopicName>/agent/camera/depth/image_raw</depthImageTopicName>
+          <depthImageCameraInfoTopicName>/agent/camera/depth/camera_info</depthImageCameraInfoTopicName>
+          <pointCloudTopicName>/agent/camera/depth/points</pointCloudTopicName>
+          <frameName>dumb_kinetic</frameName>
+          <pointCloudCutoff>0.5</pointCloudCutoff>
+          <pointCloudCutoffMax>3.0</pointCloudCutoffMax>
+          <distortionK1>0</distortionK1>
+          <distortionK2>0</distortionK2>
+          <distortionK3>0</distortionK3>
+          <distortionT1>0</distortionT1>
+          <distortionT2>0</distortionT2>
+          <CxPrime>0</CxPrime>
+          <Cx>0</Cx>
+          <Cy>0</Cy>
+          <focalLength>0</focalLength>
+          <hackBaseline>0</hackBaseline>
+      </plugin>
+    </sensor>
+  </gazebo>
 </robot>

File: robot/lidar2.xacro (robot description, xacro)
@@ -45,5 +45,5 @@
             </plugin>
             <update_rate>10</update_rate>
-            <visualize>true</visualize>
+            <visualize>false</visualize>
         </sensor>
     </gazebo>

File: robot/robot.urdf.xacro (robot description, xacro)
@@ -5,5 +5,5 @@
     <!-- <xacro:include filename="camera2.xacro"/> -->
     <!-- <xacro:include filename="depth_camera.xacro"/> -->
-    <!-- <xacro:include filename="lidar2.xacro"/> -->
+    <xacro:include filename="lidar2.xacro"/>
     <xacro:include filename="kinetic.xacro"/>
 </robot>
